File: Hardware/Estacion/Estacion.kicad_pcb (KiCad board)
At the start: 2 copper layers, 11 parts, among them J1 Screw_Terminal_01x02, J2 Step_Down_Mini

Commit message: se avanzo el PCB y ESQUEMATICO
Parts:
- added Hall1: Conn_01x03_Pin, Connector_JST:JST_PH_B3B-PH-K_1x03_P2.00mm_Vertical, F.Cu at (69.3, 28.9)
- added R1: 10K, Resistor_SMD:R_0805_2012Metric_Pad1.20x1.40mm_HandSolder, B.Cu at (79.4, 73.0)
- added R2: 10K, Resistor_SMD:R_0805_2012Metric_Pad1.20x1.40mm_HandSolder, B.Cu at (78.6, 45.3)
- added R3: 10K, Resistor_SMD:R_0805_2012Metric_Pad1.20x1.40mm_HandSolder, B.Cu at (79.3, 54.5)
- added R4: 10K, Resistor_SMD:R_0805_2012Metric_Pad1.20x1.40mm_HandSolder, B.Cu at (81.3, 63.6)
- added R5: 10K, Resistor_SMD:R_0805_2012Metric_Pad1.20x1.40mm_HandSolder, B.Cu at (75.6, 25.7)
- added R6: 10K, Resistor_SMD:R_0805_2012Metric_Pad1.20x1.40mm_HandSolder, B.Cu at (75.2, 31.5)
- added hall2: Conn_01x03_Pin, Connector_JST:JST_PH_B3B-PH-K_1x03_P2.00mm_Vertical, F.Cu at (62.6, 28.8)
- added hall_1_oeste1: Conn_01x03_Pin, Connector_JST:JST_PH_B3B-PH-K_1x03_P2.00mm_Vertical, F.Cu at (84.8, 49.5)
- added hall_2_oeste1: Conn_01x03_Pin, Connector_JST:JST_PH_B3B-PH-K_1x03_P2.00mm_Vertical, F.Cu at (84.8, 58.6)
- Aux1: renamed from Pantalla1; footprint Connector_PinSocket_2.54mm:PinSocket_1x04_P2.54mm_Vertical -> Connector_JST:JST_PH_B4B-PH-K_1x04_P2.00mm_Vertical
- BME280: footprint Connector_PinSocket_2.54mm:PinSocket_1x04_P2.54mm_Vertical -> Connector_JST:JST_PH_B4B-PH-K_1x04_P2.00mm_Vertical
- Pantalla1: renamed from Aux1; footprint Connector_PinSocket_2.54mm:PinSocket_1x04_P2.54mm_Vertical -> Connector_JST:JST_PH_B4B-PH-K_1x04_P2.00mm_Vertical
- hall_1_este1: renamed from hall_1; footprint Connector_PinHeader_2.54mm:PinHeader_1x03_P2.54mm_Vertical -> Connector_JST:JST_PH_B3B-PH-K_1x03_P2.00mm_Vertical
- hall_2_sur1: renamed from hall_2; footprint Connector_PinHeader_2.54mm:PinHeader_1x03_P2.54mm_Vertical -> Connector_JST:JST_PH_B3B-PH-K_1x03_P2.00mm_Vertical
- moved hall_1_este1 59.6 mm to (84.8, 68.0), turned to -90 degrees
- moved hall_2_sur1 43.6 mm to (84.8, 40.3), turned to -90 degrees
- moved J1 18.7 mm to (58.1, 85.3), turned to 180 degrees
- moved Aux1 11.9 mm to (48.0, 28.0), turned to -90 degrees
- moved Switc1 10.9 mm to (43.5, 75.3), turned to -90 degrees
- moved Pantalla1 10.7 mm to (40.4, 28.0), turned to -90 degrees
- moved C_0.33µF2 9.97 mm to (53.9, 70.5)
- moved J2 9.97 mm to (46.8, 81.2)
- moved C_0.33µF1 9.97 mm to (57.6, 70.5)
- moved BME280 9.82 mm to (55.7, 28.0), turned to -90 degrees
Connections:
- Esp1 pad 12: unconnected-(Esp1-IO14-Pad12) -> OUT_3
- Esp1 pad 15: unconnected-(Esp1-IO13-Pad15) -> OUT_4
- Esp1 pad 27: unconnected-(Esp1-IO16-Pad27) -> OUT_5
- Esp1 pad 28: unconnected-(Esp1-IO17-Pad28) -> OUT_6
Routing:
- net 3V3: track 0.00 -> 66.2 mm, vias 0 -> 1
- net VO+: track 4.80 -> 66.3 mm
- net OUT_2: track 0.00 -> 52.7 mm
- net OUT_3: track 0.00 -> 41.1 mm
- net SCL: track 0.00 -> 31.1 mm
- net Net-(J1-Pin_2): track 0.00 -> 29.5 mm
- net OUT_4: track 0.00 -> 24.5 mm
- net SDA: track 0.00 -> 22.1 mm
- net GND: track 0.00 -> 15.2 mm
- net VIN+: track 5.10 -> 11.5 mm
- net OUT_1: track 0.00 -> 5.35 mm

Commit message: Primera version del PCB
Parts:
- removed Switc1: SW_SPDT, EESTN5:SW_SPDT_TH_100Mils_VERTICAL
- added J3: Conn_01x03_Pin, Connector_JST:JST_PH_B3B-PH-K_1x03_P2.00mm_Vertical, F.Cu at (43.0, 76.1)
- moved J1 23.4 mm to (35.1, 81.1), turned to 90 degrees
- moved R6 16.2 mm to (60.7, 24.2), turned to 180 degrees
- moved R5 5.88 mm to (69.9, 24.4), turned to 180 degrees
- moved hall2 4.92 mm to (57.7, 28.0), turned to 0 degrees
- moved R4 3.36 mm to (78.6, 61.6), turned to 90 degrees
- moved C_0.33µF1 3.29 mm to (57.1, 73.7)
- moved C_0.33µF2 3.29 mm to (53.4, 73.7)
- moved J2 3.29 mm to (46.3, 84.5)
- moved BME280 3.24 mm to (52.4, 28.0)
- moved Hall1 2.61 mm to (66.9, 28.0), turned to 0 degrees
- moved Aux1 1.63 mm to (46.4, 28.0)
- moved R1 0.81 mm to (78.6, 73.0)
- moved R3 0.71 mm to (78.6, 54.5)
Connections:
- Esp1 pad 14: unconnected-(Esp1-GND-Pad14) -> GND
- Esp1 pad 32: unconnected-(Esp1-GND-Pad32) -> GND
- Esp1 pad 38: unconnected-(Esp1-GND-Pad38) -> GND
Routing:
- net 3V3: track 66.2 -> 238.8 mm, vias 1 -> 6
- net VO+: track 66.3 -> 187.6 mm
- net OUT_1: track 5.35 -> 38.8 mm
- net OUT_5: track 0.00 -> 26.7 mm
- net OUT_6: track 0.00 -> 20.2 mm
- net Net-(J1-Pin_2): track 29.5 -> 10.0 mm
- net GND: track 15.2 -> 0.00 mm
- net SDA: track 22.1 -> 18.8 mm
- net SCL: track 31.1 -> 27.9 mm
- added copper zone on B.Cu, net GND
